Commit message: URDF changed for x along the length of the robot, and angle computation also changed

File: src/myrobot_gazebo/urdf/myrobot_descr (copy).xacro (robot description, xacro)
@@ -21,5 +21,5 @@
    		<visual>
      			<geometry>
-       				<box size="0.3 0.2 0.1"/>
+       				<box size="0.2 0.3 0.1"/>
      			</geometry>
 			<origin rpy="0 0 0" xyz="0 0 0.05"/>
@@ -30,5 +30,5 @@
 		<collision>
 			<geometry>
-       				<box size="0.3 0.2 0.1"/>
+       				<box size="0.2 0.3 0.1"/>
 			</geometry>
 		</collision>
@@ -38,5 +38,5 @@
    		<visual>
      			<xacro:wheel_geometry />
-			<origin rpy="0 1.5707 1.5707" xyz="0.0 0.0 0"/>
+			<origin rpy="0 1.5707 0" xyz="0.0 0.0 0"/>
    			<material name="black">
 				<color rgba="0 0 0 1"/>
@@ -51,5 +51,5 @@
    		<visual>
      			<xacro:wheel_geometry />
-			<origin rpy="0 1.5707 1.5707" xyz="-0.0 0.0 0"/>
+			<origin rpy="0 1.5707 0" xyz="-0.0 0.0 0"/>
    			<material name="black"/>
    		</visual>
@@ -62,5 +62,5 @@
    		<visual>
  			<xacro:wheel_geometry />
-			<origin rpy="0 1.5707 1.5707" xyz="0.0 -0.0 0"/>
+			<origin rpy="0 1.5707 0" xyz="0.0 -0.0 0"/>
    			<material name="black"/>
    		</visual>
@@ -73,5 +73,5 @@
    		<visual>
   			 <xacro:wheel_geometry />
-			<origin rpy="0 1.5707 1.5707" xyz="-0.0 -0.0 0"/>
+			<origin rpy="0 1.5707 0" xyz="-0.0 -0.0 0"/>
    			<material name="black"/>
    		</visual>
@@ -107,6 +107,6 @@
 <!-- CAMERA -->
 	 <joint name="camera_joint" type="fixed">
-	    <axis xyz="-1 0 0" />
-	    <origin xyz="0.125 0 0.125" rpy="0 0 0"/>
+	    <axis xyz="0 1 0" />
+	    <origin xyz="0 0.125 0.125" rpy="0 0 1.57"/>
 	    <parent link="base_link"/>
 	    <child link="camera_link"/>
