Commit message: URDF updated

File: src/myrobot_gazebo/urdf/myrobot_descr.xacro (robot description, xacro)
@@ -3,6 +3,6 @@
 <xacro:include filename="$(find myrobot_gazebo)/urdf/myrobot_descr.gazebo"/>
 <!-- ROBOT -->
-	<xacro:property name="length_wheel" value="0.05" />
-	<xacro:property name="radius_wheel" value="0.05" />
+	<xacro:property name="length_wheel" value="0.036" />
+	<xacro:property name="radius_wheel" value="0.04" />
 	<xacro:macro name="default_inertial" params="mass">
                <inertial>
@@ -21,7 +21,7 @@
    		<visual>
      			<geometry>
-       				<box size="0.3 0.2 0.1"/>
+       				<box size="0.205 0.155 0.02"/>
      			</geometry>
-			<origin rpy="0 0 0" xyz="0 0 0.05"/>
+			<origin rpy="0 0 0" xyz="0 0 0.04"/>
 			<material name="white">
 				<color rgba="1 1 1 1"/>
@@ -30,8 +30,8 @@
 		<collision>
 			<geometry>
-       				<box size="0.3 0.2 0.1"/>
+       				<box size="0.205 0.155 0.02"/>
 			</geometry>
 		</collision>
-		<xacro:default_inertial mass="10"/>
+		<xacro:default_inertial mass="1"/>
  	</link>
  	<link name="wheel_1">
@@ -46,5 +46,5 @@
 			<xacro:wheel_geometry />
 		</collision>
-		<xacro:default_inertial mass="1"/>
+		<xacro:default_inertial mass="0.01"/>
  	</link>
  	<link name="wheel_2">
@@ -57,5 +57,5 @@
 			<xacro:wheel_geometry />
 		</collision>
-		<xacro:default_inertial mass="1"/>
+		<xacro:default_inertial mass="0.01"/>
  	</link>
  	<link name="wheel_3">
@@ -68,5 +68,5 @@
 			<xacro:wheel_geometry />
 		</collision>
-		<xacro:default_inertial mass="1"/>
+		<xacro:default_inertial mass="0.01"/>
  	</link>
  	<link name="wheel_4">
@@ -79,5 +79,5 @@
 			<xacro:wheel_geometry />
 		</collision>
-		<xacro:default_inertial mass="1"/>
+		<xacro:default_inertial mass="0.01"/>
  	</link>
  	<joint name="base_to_wheel1" type="continuous">
@@ -85,5 +85,5 @@
 		<child link="wheel_1"/>
                 <axis xyz="1 0 0"/>
-		<origin xyz="0.1 0.1 0"/>
+		<origin xyz="0.05 0.098 0.04"/>
 	</joint>
 	<joint name="base_to_wheel2" type="continuous">
@@ -91,5 +91,5 @@
 		<child link="wheel_2"/>
                 <axis xyz="1 0 0"/>
-		<origin xyz="-0.1 0.1 0"/>
+		<origin xyz="-0.05 0.098 0.04"/>
 	</joint>
 	<joint name="base_to_wheel3" type="continuous">
@@ -97,5 +97,5 @@
 		<child link="wheel_3"/>
                 <axis xyz="1 0 0"/>
-		<origin xyz="0.1 -0.1 0"/>
+		<origin xyz="0.05 -0.098 0.04"/>
 	</joint>
 	<joint name="base_to_wheel4" type="continuous">
@@ -103,10 +103,10 @@
 		<child link="wheel_4"/>
                 <axis xyz="1 0 0"/>
-		<origin xyz="-0.1 -0.1 0"/>
+		<origin xyz="-0.05 -0.098 0.04"/>
 	</joint>
 <!-- CAMERA -->
 	 <joint name="camera_joint" type="fixed">
 	    <axis xyz="-1 0 0" />
-	    <origin xyz="0.125 0 0.125" rpy="0 0 0"/>
+	    <origin xyz="0.090 0 0.06" rpy="0 0 0"/>
 	    <parent link="base_link"/>
 	    <child link="camera_link"/>
@@ -116,5 +116,5 @@
 	      <origin xyz="0 0 0" rpy="0 0 0"/>
 	      <geometry>
-		<box size="0.05 0.05 0.05"/>
+		<box size="0.01 0.05 0.05"/>
 	      </geometry>
 	    </collision>
@@ -122,5 +122,5 @@
 	      <origin xyz="0 0 0" rpy="0 0 0"/>
 	      <geometry>
-		<box size="0.05 0.05 0.05"/>
+		<box size="0.01 0.05 0.05"/>
 	      </geometry>
 	      <material name="red">
